File: hardware/v1/v1.kicad_pcb (KiCad board)
At the start: 2 copper layers, 54 x 86 mm, 36 parts, among them J1 FPC 24P 0.5mm bottom contact, J2 UP port, JST-SH 4, J3 DN port, JST-SH 4, J4 UP, magnetic pogo pins, J5 Qwiic / STEMMA QT, JST-SH 4, J6 spare GPIO, 2x5, M1 5x2 mm disc, M2 5x2 mm disc, M3 5x2 mm disc, M4 5x2 mm disc, P1 DN, magnetic pads, in the tra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, Q1 AO3400A, SW1 power, SW2 A: next, SW3 B: confirm, U1 Raspberry Pi Pico 2 (no heade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

Commit message: V1 board: the NXP SE051 secure element on I2C0 with a three-turn NFC loop around the board's perimeter, a slide switch in the antenna line and tuning capacitors; a 10-pin JST-SH expansion socket in place of the 2x5 header; sockets turned to open at the edge; BOM part numbers verified against JLCPCB's stock (the 2.2 ohm sense resistor was a 22 ohm code); escape stubs for the chip's 0.4 mm pitch; the panel taped to the board and the tray with switch openings; quoted through ProvenMetal. Pico 2 firmware: latched peer detection, preallocated link queues, 115200 baud with the RX trigger at 1/8, and a boot probe that gets an R-block back from the SE051 Click board
Parts:
- added ANT1: NFC loop, 4 turns, cahoots:NFC_loop, F.Cu at (126.0, 64.5)
- added C13: 100nF 50V, C_0603_1608Metric, B.Cu at (107.0, 67.0)
- added C14: 100nF 50V, C_0603_1608Metric, B.Cu at (107.0, 70.0)
- added C15: 39pF C0G, C_0603_1608Metric, B.Cu at (111.5, 67.0)
- added C16: 27pF C0G, C_0603_1608Metric, B.Cu at (115.5, 67.0)
- added R3: 3.3k, R_0603_1608Metric, B.Cu at (86.0, 75.0)
- added R4: 3.3k, R_0603_1608Metric, B.Cu at (86.0, 72.0)
- added R5: 100k, R_0603_1608Metric, B.Cu at (120.5, 68.0)
- added SW4: antenna, SW_SPDT_Shouhan_MSK12C02, B.Cu at (121.0, 74.6)
- added U2: SE051C2, QFN-20-1EP_3x3mm_P0.4mm_EP1.65x1.65mm, B.Cu at (111.5, 73.5)
- J6: value spare GPIO, 2x5 -> expansion, JST-SH 10; footprint PinHeader_2x05_P2.54mm_Vertical -> JST_SH_SM10B-SRSS-TB_1x10-1MP_P1.00mm_Horizontal
- moved J6 7.68 mm to (100.0, 139.5)
- moved D4 7.52 mm to (86.5, 137.5)
- turned J2 to 0 degrees
- turned J3 to 0 degrees
- turned J5 to 0 degrees
Connections:
- U1 pad 4: (no net) -> SE_ENA
Routing:
- net 3V3: track 80.5 -> 168.3 mm, vias 1 -> 5
- net SE_ENA: track 0.00 -> 50.3 mm
- net LA: track 0.00 -> 39.6 mm
- net GP26: track 37.0 -> 65.1 mm, vias 1 -> 2
- net I2C_SDA: track 78.1 -> 102.5 mm, vias 5 -> 4
- net LB: track 0.00 -> 24.0 mm, vias 0 -> 2
- net SE_VCC: track 0.00 -> 23.8 mm, vias 0 -> 3
- net I2C_SCL: track 79.0 -> 102.2 mm, vias 5 -> 3
- net GP22: track 32.8 -> 54.9 mm, vias 1 -> 4
- net ANT: track 0.00 -> 14.6 mm
- net EPD_DC: track 44.9 -> 58.2 mm
- net VGL: track 25.9 -> 13.7 mm
- net GP13: track 58.7 -> 70.5 mm, vias 1 -> 4
- net DN_RX: track 69.9 -> 81.1 mm, vias 1 -> 3
- net GP11: track 56.4 -> 67.1 mm, vias 1 -> 4
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