File: hardware/v1/v1.kicad_sch (KiCad schematic)
At the start: 29 parts, among them J1 FPC 24P 0.5mm bottom contact, J2 UP port, JST-SH 4, J3 DN port, JST-SH 4, J4 UP, magnetic pogo pins, J5 Qwiic / STEMMA QT, JST-SH 4, J6 spare GPIO, 2x5, Q1 AO3400A, SW1 power, SW2 A: next, SW3 B: confirm, U1 Raspberry Pi Pico 2 (no heade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

Commit message: V1 board: the NXP SE051 secure element on I2C0 with a three-turn NFC loop around the board's perimeter, a slide switch in the antenna line and tuning capacitors; a 10-pin JST-SH expansion socket in place of the 2x5 header; sockets turned to open at the edge; BOM part numbers verified against JLCPCB's stock (the 2.2 ohm sense resistor was a 22 ohm code); escape stubs for the chip's 0.4 mm pitch; the panel taped to the board and the tray with switch openings; quoted through ProvenMetal. Pico 2 firmware: latched peer detection, preallocated link queues, 115200 baud with the RX trigger at 1/8, and a boot probe that gets an R-block back from the SE051 Click board
Parts:
- removed J6: spare GPIO, 2x5, Connector_PinHeader_2.54mm:PinHeader_2x05_P2.54mm_Vertical, symbol Connector_Generic:Conn_02x05_Odd_Even
- added ANT1: NFC loop, 4 turns, cahoots:NFC_loop, symbol Device:Antenna_Loop
- added C13, C14: 100nF 50V, Capacitor_SMD:C_0603_1608Metric, symbol Device:C
- added C15: 39pF C0G, Capacitor_SMD:C_0603_1608Metric, symbol Device:C
- added C16: 27pF C0G, Capacitor_SMD:C_0603_1608Metric, symbol Device:C
- added J6: expansion, JST-SH 10, Connector_JST:JST_SH_SM10B-SRSS-TB_1x10-1MP_P1.00mm_Horizontal, symbol Connector_Generic:Conn_01x10
- added R3, R4: 3.3k, Resistor_SMD:R_0603_1608Metric, symbol Device:R
- added R5: 100k, Resistor_SMD:R_0603_1608Metric, symbol Device:R
- added SW4: antenna, Button_Switch_SMD:SW_SPDT_Shouhan_MSK12C02, symbol Switch:SW_SPDT
- added U2: SE051C2, Package_DFN_QFN:QFN-20-1EP_3x3mm_P0.4mm_EP1.65x1.65mm, symbol cahoots:SE051
- BT1: LCSC MYOUNG BS-07-A1BJ001 (LCSC number to confirm) -> C2979167 MYOUNG BS-07-A1BJ001
- L1: LCSC FNR4030S470MT (verify) -> C167888 FNR4030S470MT
- R2: LCSC C23345 (verify) -> C22939 0603WAF220KT5E, 2.2 ohm
- SW2, SW3: LCSC C318884 -> C318884 TS-1187A-B-A-B
- U1: LCSC consigned: solder by hand -> not fitted: solder by hand
Connections:
- net 3V3: now also C13.1, J6.1 (Pin_1), R3.2, R4.2, R5.2, U2.12 (VIN)
- net GND: now also C13.2, C14.2, J6.2 (Pin_2), U2.19 (VSS)
- net GP10: now also J6.5 (Pin_5)
- net GP11: now also J6.6 (Pin_6)
- net GP12: now also J6.7 (Pin_7)
- net GP13: now also J6.8 (Pin_8)
- net GP22: now also J6.9 (Pin_9)
- net GP26: now also J6.10 (Pin_10)
- net GP6: now also J6.3 (Pin_3)
- net GP7: now also J6.4 (Pin_4)
- net I2C_SCL: now also R4.1, U2.10 (SCL)
- net I2C_SDA: now also R3.1, U2.9 (SDA)
- net SE_ENA: now reaches U1.4 (GP2)
- net SE_ENA: now also R5.1, U2.11 (ENA)
- new net ANT: ANT1.1, SW4.2 (B)
- new net LA: C15.1, C16.1, SW4.1 (A), U2.17 (LA)
- new net LB: ANT1.2, C15.2, C16.2, U2.1 (LB)
- new net SE_VCC: C14.1, U2.14 (RST_N), U2.15 (VOUT), U2.18 (VCC)
- no-connect marks 17 -> 28
Other:
- note added: "Antenna: C15 (27 pF) and C16 (not fitted, trim) across LA/LB at the chip, SW4 opens the LA line, ANT1 is the four-turn loop on the front."
- note added: "Secure element: NXP SE051 on I2C0. ENA low is deep power-down; R5 holds it on. VOUT ties to VCC (SE_VCC), as the data sheet asks when ENA is used."
